File: libraries/PU2CLR_SI4735/extras/schematic/schematic_esp32_lcd_16x2_OR_lcd20x4.sch (EAGLE design)
At the start: 22 parts, among them U1 SI4735-D60-GU, U2 ESP32-DEVKITC-32D

Commit message: updates
Parts:
- removed R4: 2K, adafruit:R-US_0204/2V
- added VR1: 10k, SparkFun-Resistors:POTENTIOMETER-PTH-9MM-1/20W-20%
Connections:
- net GND: now also VR1.A; no longer R4.2
- net N$21: now also VR1.S; no longer R4.1
- net VCC: now also VR1.E
Other:
- note added: "GPIO15"
- note added: "GPIO16"
- note added: "GPIO17"
- note added: "GPIO18"
- note added: "LCD 20x4 or 16x2"
- note removed: "LCD 20x4"
- moved on the sheet: R1, R2, S2
